Commit message: Added MuJoCo pick and place demo with default trajectory

File: install/robotic_arm_model_v3/share/robotic_arm_model_v3/urdf/robotic_arm_model_v3.urdf (robot description, URDF)
Before this commit: robot robotic_arm_model_v3, 9 links, 8 joints
Joints:
- joint joint_1: origin xyz=0.681512899942898 -1.31957371207269 0.9106277233023 rpy=1.57079632679489 0 2.30611320700167 -> xyz=0 0 0 rpy=1.57079632679489 0 2.30611320700167

File: install/robotic_arm_v3_config/share/robotic_arm_v3_config/config/robotic_arm_model_v3.ros2_control.xacro (robot description, xacro)
@@ -1,39 +1,34 @@
 <?xml version="1.0"?>
 <robot xmlns:xacro="http://www.ros.org/wiki/xacro">
-    <xacro:macro name="robotic_arm_model_v3_ros2_control" params="name initial_positions_file">
+    <xacro:macro name="robotic_arm_model_v3_ros2_control" params="name initial_positions_file use_sim:=false headless:=false">
         <xacro:property name="initial_positions" value="${xacro.load_yaml(initial_positions_file)['initial_positions']}"/>
         <ros2_control name="${name}" type="system">
             <hardware>
-                <!-- By default, set up controllers for simulation. This won't work on real hardware -->
-                <plugin>mock_components/GenericSystem</plugin>
+                <xacro:if value="${use_sim == 'mujoco'}">
+                    <plugin>mujoco_ros2_control/MujocoSystemInterface</plugin>
+                    <param name="mujoco_model">$(find robotic_arm_v3_config)/config/mujoco/arm_scene.xml</param>
+                    <param name="headless">${headless}</param>
+                    <param name="sim_speed_factor">1.0</param>
+                </xacro:if>
+                <xacro:if value="${use_sim == 'gazebo'}">
+                    <plugin>gz_ros2_control/GazeboSimSystem</plugin>
+                </xacro:if>
+                <xacro:if value="${use_sim == 'false' or use_sim == False}">
+                    <plugin>mock_components/GenericSystem</plugin>
+                </xacro:if>
             </hardware>
-            <joint name="joint_1">
-                <command_interface name="position"/>
-                <state_interface name="position">
-                  <param name="initial_value">${initial_positions['joint_1']}</param>
-                </state_interface>
-                <state_interface name="velocity"/>
-            </joint>
-            <joint name="joint_2">
-                <command_interface name="position"/>
-                <state_interface name="position">
-                  <param name="initial_value">${initial_positions['joint_2']}</param>
-                </state_interface>
-                <state_interface name="velocity"/>
-            </joint>
-            <joint name="joint_3">
-                <command_interface name="position"/>
-                <state_interface name="position">
-                  <param name="initial_value">${initial_positions['joint_3']}</param>
-                </state_interface>
-                <state_interface name="velocity"/>
-            </joint>
-            <joint name="joint_4">
-                <command_interface name="position"/>
-                <state_interface name="position">
-                  <param name="initial_value">${initial_positions['joint_4']}</param>
-                </state_interface>
-                <state_interface name="velocity"/>
-            </joint>
+            <xacro:macro name="configure_joint" params="joint_name">
+                <joint name="${joint_name}">
+                    <command_interface name="position"/>
+                    <state_interface name="position">
+                      <param name="initial_value">${initial_positions[joint_name]}</param>
+                    </state_interface>
+                    <state_interface name="velocity"/>
+                </joint>
+            </xacro:macro>
+            <xacro:configure_joint joint_name="joint_1"/>
+            <xacro:configure_joint joint_name="joint_2"/>
+            <xacro:configure_joint joint_name="joint_3"/>
+            <xacro:configure_joint joint_name="joint_4"/>
             <joint name="end_effector_joint">
                 <command_interface name="position"/>

File: install/robotic_arm_v3_config/share/robotic_arm_v3_config/config/robotic_arm_model_v3.urdf.xacro (robot description, xacro)
@@ -2,8 +2,31 @@
 <robot xmlns:xacro="http://www.ros.org/wiki/xacro" name="robotic_arm_model_v3">
     <xacro:arg name="initial_positions_file" default="initial_positions.yaml" />
+    <!-- use_sim: mujoco → mujoco_ros2_control/MujocoSystemInterface
+                 gazebo → gz_ros2_control/GazeboSimSystem + Gazebo plugin
+                 false  → mock_components/GenericSystem (MoveIt-only sim) -->
+    <xacro:arg name="use_sim" default="false" />
+    <xacro:arg name="headless" default="false" />
     <!-- Import robotic_arm_model_v3 urdf file -->
     <xacro:include filename="$(find robotic_arm_model_v3)/urdf/robotic_arm_model_v3.urdf" />
     <!-- Import control_xacro -->
     <xacro:include filename="robotic_arm_model_v3.ros2_control.xacro" />
-    <xacro:robotic_arm_model_v3_ros2_control name="FakeSystem" initial_positions_file="$(arg initial_positions_file)"/>
+    <xacro:robotic_arm_model_v3_ros2_control
+        name="ArmSystem"
+        initial_positions_file="$(arg initial_positions_file)"
+        use_sim="$(arg use_sim)"
+        headless="$(arg headless)"/>
+    <!-- When running in Gazebo, inject the gz_ros2_control system plugin.
+         The <gazebo> tag is converted to a <plugin> element in the SDF
+         that Gazebo loads when it spawns the robot from robot_description. -->
+    <xacro:if value="${'$(arg use_sim)' == 'gazebo'}">
+        <gazebo>
+            <plugin filename="gz_ros2_control-system"
+                    name="gz_ros2_control::GazeboSimROS2ControlPlugin">
+                <parameters>$(find robotic_arm_v3_config)/config/ros2_controllers.yaml</parameters>
+                <ros>
+                    <namespace>/</namespace>
+                </ros>
+            </plugin>
+        </gazebo>
+    </xacro:if>
 </robot>
